Commit message: tf read

File: urdf/model.urdf (robot description, URDF)
Before this commit: robot parallel_car, 8 links, 7 joints
Links:
- added link down_1, mass 0.01; visual box size=0.001 0.001 0.001
- added link down_1_medium, mass 0.01; visual box size=0.001 0.001 0.001
- added link down_2, mass 0.01; visual box size=0.001 0.001 0.001
- added link down_2_medium, mass 0.01; visual box size=0.001 0.001 0.001
- added link down_3, mass 0.01; visual box size=0.001 0.001 0.001
- added link down_3_medium, mass 0.01; visual box size=0.001 0.001 0.001
- added link down_4, mass 0.01; visual box size=0.001 0.001 0.001
- added link down_4_medium, mass 0.01; visual box size=0.001 0.001 0.001
- added link down_5, mass 0.01; visual box size=0.001 0.001 0.001
- added link down_5_medium, mass 0.01; visual box size=0.001 0.001 0.001
- added link down_6, mass 0.01; visual box size=0.001 0.001 0.001
- added link down_6_medium, mass 0.01; visual box size=0.001 0.001 0.001
- added link down_link, mass 0.5; collision mesh filename=package://parallel_car/meshes/platform_down.STL; visual mesh filename=package://parallel_car/meshes/platform_down.STL
- added link up_1, mass 0.01; visual box size=0.001 0.001 0.001
- added link up_1_medium, mass 0.01; visual box size=0.001 0.001 0.001
- added link up_2, mass 0.01; visual box size=0.001 0.001 0.001
- added link up_2_medium, mass 0.01; visual box size=0.001 0.001 0.001
- added link up_3, mass 0.01; visual box size=0.001 0.001 0.001
- added link up_3_medium, mass 0.01; visual box size=0.001 0.001 0.001
- added link up_4, mass 0.01; visual box size=0.001 0.001 0.001
- added link up_4_medium, mass 0.01; visual box size=0.001 0.001 0.001
- added link up_5, mass 0.01; visual box size=0.001 0.001 0.001
- added link up_5_medium, mass 0.01; visual box size=0.001 0.001 0.001
- added link up_6, mass 0.01; visual box size=0.001 0.001 0.001
- added link up_6_medium, mass 0.01; visual box size=0.001 0.001 0.001
- added link up_link, mass 0.3; collision mesh filename=package://parallel_car/meshes/platform_up.STL; visual mesh filename=package://parallel_car/meshes/platform_up.STL
- link car_link: geometry collision box size=1 0.5 0.36; visual box size=1 0.5 0.36
Joints:
- added joint car_to_down: type fixed, parent car_link, child down_link, origin xyz=0.0 0.0 0.18 rpy=0.0 0.0 0.0
- added joint littleY_to_up: type fixed, parent littleY_link, child up_link, origin xyz=0.0 0.0 0.0 rpy=0.0 0.0 0.0
- added joint medium_to_down_1: type fixed, parent down_1_medium, child down_1, origin xyz=0.2 0.0 0.075 rpy=0.0 0.0 0.0
- added joint medium_to_down_2: type fixed, parent down_2_medium, child down_2, origin xyz=0.2 0.0 0.075 rpy=0.0 0.0 0.0
- added joint medium_to_down_3: type fixed, parent down_3_medium, child down_3, origin xyz=0.2 0.0 0.075 rpy=0.0 0.0 0.0
- added joint medium_to_down_4: type fixed, parent down_4_medium, child down_4, origin xyz=0.2 0.0 0.075 rpy=0.0 0.0 0.0
- added joint medium_to_down_5: type fixed, parent down_5_medium, child down_5, origin xyz=0.2 0.0 0.075 rpy=0.0 0.0 0.0
- added joint medium_to_down_6: type fixed, parent down_6_medium, child down_6, origin xyz=0.2 0.0 0.075 rpy=0.0 0.0 0.0
- added joint medium_to_up_1: type fixed, parent up_1_medium, child up_1, origin xyz=0.1 0.0 -0.05 rpy=0.0 0.0 0.0
- added joint medium_to_up_2: type fixed, parent up_2_medium, child up_2, origin xyz=0.1 0.0 -0.05 rpy=0.0 0.0 0.0
- added joint medium_to_up_3: type fixed, parent up_3_medium, child up_3, origin xyz=0.1 0.0 -0.05 rpy=0.0 0.0 0.0
- added joint medium_to_up_4: type fixed, parent up_4_medium, child up_4, origin xyz=0.1 0.0 -0.05 rpy=0.0 0.0 0.0
- added joint medium_to_up_5: type fixed, parent up_5_medium, child up_5, origin xyz=0.1 0.0 -0.05 rpy=0.0 0.0 0.0
- added joint medium_to_up_6: type fixed, parent up_6_medium, child up_6, origin xyz=0.1 0.0 -0.05 rpy=0.0 0.0 0.0
- added joint up_to_down_1_medium: type fixed, parent down_link, child down_1_medium, origin xyz=0.0 0.0 0.0 rpy=0.0 0.0 0.174532925199
- added joint up_to_down_2_medium: type fixed, parent down_link, child down_2_medium, origin xyz=0.0 0.0 0.0 rpy=0.0 0.0 1.91986217719
- added joint up_to_down_3_medium: type fixed, parent down_link, child down_3_medium, origin xyz=0.0 0.0 0.0 rpy=0.0 0.0 2.26892802759
- added joint up_to_down_4_medium: type fixed, parent down_link, child down_4_medium, origin xyz=0.0 0.0 0.0 rpy=0.0 0.0 4.01425727959
- added joint up_to_down_5_medium: type fixed, parent down_link, child down_5_medium, origin xyz=0.0 0.0 0.0 rpy=0.0 0.0 4.36332312999
- added joint up_to_down_6_medium: type fixed, parent down_link, child down_6_medium, origin xyz=0.0 0.0 0.0 rpy=0.0 0.0 6.10865238198
- added joint up_to_up_1_medium: type fixed, parent up_link, child up_1_medium, origin xyz=0.0 0.0 0.0 rpy=0.0 0.0 0.872664625997
- added joint up_to_up_2_medium: type fixed, parent up_link, child up_2_medium, origin xyz=0.0 0.0 0.0 rpy=0.0 0.0 1.2217304764
- added joint up_to_up_3_medium: type fixed, parent up_link, child up_3_medium, origin xyz=0.0 0.0 0.0 rpy=0.0 0.0 2.96705972839
- added joint up_to_up_4_medium: type fixed, parent up_link, child up_4_medium, origin xyz=0.0 0.0 0.0 rpy=0.0 0.0 3.31612557879
- added joint up_to_up_5_medium: type fixed, parent up_link, child up_5_medium, origin xyz=0.0 0.0 0.0 rpy=0.0 0.0 5.06145483078
- added joint up_to_up_6_medium: type fixed, parent up_link, child up_6_medium, origin xyz=0.0 0.0 0.0 rpy=0.0 0.0 5.41052068118

File: urdf/parallel_car.urdf.xacro (robot description, xacro)
@@ -5,4 +5,5 @@
     <xacro:include filename="$(find parallel_car)/urdf/parallel_car.transmission.xacro"/>
     <xacro:include filename="$(find parallel_car)/urdf/materials.xacro"/>
+    <xacro:include filename="$(find parallel_car)/urdf/sub_link.urdf.xacro"/>
     <!--xacro properties-->
     <xacro:property name="car_mass" value="20.0"/>
@@ -14,4 +15,9 @@
     <xacro:property name="little_width" value="0.001"/>
     <xacro:property name="wx_length" value="0.55"/>
+    <xacro:property name="down_radius" value="0.2"/>
+    <xacro:property name="down_height" value="0.075"/>
+    <xacro:property name="up_radius" value="0.1"/>
+    <xacro:property name="up_height" value="0.05"/>
+    <xacro:property name="little_mass" value="0.01"/>
     <!-- links -->
     <link name="car_link"><!--from origin to top-->
@@ -235,3 +241,16 @@
         <child link="up_link"/>
     </joint>
+    <!-- spawn the sub links and joints-->
+    <xacro:sub_link_joint parent_link="down_link" child_link="down_1" height="${down_height}" radius="${down_radius}" beta="10.0" little_width="${little_width}" little_mass="${little_mass}" />
+    <xacro:sub_link_joint parent_link="down_link" child_link="down_2" height="${down_height}" radius="${down_radius}" beta="110.0" little_width="${little_width}" little_mass="${little_mass}" />
+    <xacro:sub_link_joint parent_link="down_link" child_link="down_3" height="${down_height}" radius="${down_radius}" beta="130.0" little_width="${little_width}" little_mass="${little_mass}" />
+    <xacro:sub_link_joint parent_link="down_link" child_link="down_4" height="${down_height}" radius="${down_radius}" beta="230.0" little_width="${little_width}" little_mass="${little_mass}" />
+    <xacro:sub_link_joint parent_link="down_link" child_link="down_5" height="${down_height}" radius="${down_radius}" beta="250.0" little_width="${little_width}" little_mass="${little_mass}" />
+    <xacro:sub_link_joint parent_link="down_link" child_link="down_6" height="${down_height}" radius="${down_radius}" beta="350.0" little_width="${little_width}" little_mass="${little_mass}" />
+    <xacro:sub_link_joint parent_link="up_link" child_link="up_1" height="${up_height}" radius="${up_radius}" beta="50.0" little_width="${little_width}" little_mass="${little_mass}" />
+    <xacro:sub_link_joint parent_link="up_link" child_link="up_2" height="${up_height}" radius="${up_radius}" beta="70.0" little_width="${little_width}" little_mass="${little_mass}" />
+    <xacro:sub_link_joint parent_link="up_link" child_link="up_3" height="${up_height}" radius="${up_radius}" beta="170.0" little_width="${little_width}" little_mass="${little_mass}" />
+    <xacro:sub_link_joint parent_link="up_link" child_link="up_4" height="${up_height}" radius="${up_radius}" beta="190.0" little_width="${little_width}" little_mass="${little_mass}" />
+    <xacro:sub_link_joint parent_link="up_link" child_link="up_5" height="${up_height}" radius="${up_radius}" beta="290.0" little_width="${little_width}" little_mass="${little_mass}" />
+    <xacro:sub_link_joint parent_link="up_link" child_link="up_6" height="${up_height}" radius="${up_radius}" beta="310.0" little_width="${little_width}" little_mass="${little_mass}" />
 </robot>
