Commit message: add platform stl

File: urdf/materials.xacro (robot description, xacro)
@@ -28,3 +28,6 @@
     <color rgba="1.0 1.0 0.0 1.0"/>
   </material>
+  <material name="chocolate">
+    <color rgba="${210/255} ${105/255} ${30/255} 1.0"/>
+  </material>
 </robot>

File: urdf/parallel_car.urdf.xacro (robot description, xacro)
@@ -135,4 +135,44 @@
     </link>
     <!-- up and down links -->
+    <link name="down_link">
+        <inertial>
+            <origin xyz="0.0 0.0 0.0" rpy="${PI/2.0} 0.0 ${PI/2.0}"/>
+            <mass value="0.5"/>
+            <inertia ixx="0.5" ixy="0.0" ixz="0.0" iyy="0.5" iyz="0.0" izz="0.5"/>
+        </inertial>
+        <visual>
+            <origin xyz="0.0 0.0 0.0" rpy="${PI/2.0} 0.0 ${PI/2.0}"/>
+            <geometry>
+                <mesh filename="package://parallel_car/meshes/platform_down.STL" />
+            </geometry>
+            <material name="chocolate"/>
+        </visual>
+        <collision>
+            <origin xyz="0.0 0.0 0.0" rpy="${PI/2.0} 0.0 ${PI/2.0}"/>
+            <geometry>
+                <mesh filename="package://parallel_car/meshes/platform_down.STL" />
+            </geometry>
+        </collision>
+    </link>
+    <link name="up_link">
+        <inertial>
+            <origin xyz="0.0 0.0 0.0" rpy="${-PI/2.0} 0.0 ${-PI/6.0}"/>
+            <mass value="0.3"/>
+            <inertia ixx="0.3" ixy="0.0" ixz="0.0" iyy="0.3" iyz="0.0" izz="0.3"/>
+        </inertial>
+        <visual>
+            <origin xyz="0.0 0.0 0.0" rpy="${-PI/2.0} 0.0 ${-PI/6.0}"/>
+            <geometry>
+                <mesh filename="package://parallel_car/meshes/platform_up.STL" />
+            </geometry>
+            <material name="orange"/>
+        </visual>
+        <collision>
+            <origin xyz="0.0 0.0 0.0" rpy="${-PI/2.0} 0.0 ${-PI/6.0}"/>
+            <geometry>
+                <mesh filename="package://parallel_car/meshes/platform_up.STL" />
+            </geometry>
+        </collision>
+    </link>
     <!-- joints -->
     <joint name="car_to_barX" type="prismatic">
@@ -184,8 +224,13 @@
     </joint>
     <!-- up and down joints -->
-    <!--joint name="car_to_down" type="fixed">
+    <joint name="car_to_down" type="fixed">
         <origin xyz="0.0 0.0 0.18" rpy="0.0 0.0 0.0"/>
         <parent link="car_link"/>
         <child link="down_link"/>
-    </joint-->
+    </joint>
+    <joint name="littleY_to_up" type="fixed">
+        <origin xyz="0.0 0.0 0.0" rpy="0.0 0.0 0.0"/>
+        <parent link="littleY_link"/>
+        <child link="up_link"/>
+    </joint>
 </robot>

Commit message: add tilt support to urdf

File: urdf/materials.xacro (robot description, xacro)
@@ -31,3 +31,6 @@
     <color rgba="${210/255} ${105/255} ${30/255} 1.0"/>
   </material>
+  <material name="purple">
+    <color rgba="${128/255} 0.0 ${128/255} 1.0"/>
+  </material>
 </robot>

File: urdf/parallel_car.urdf.xacro (robot description, xacro)
@@ -20,4 +20,6 @@
     <xacro:property name="up_height" value="0.05"/>
     <xacro:property name="little_mass" value="0.01"/>
+    <xacro:property name="addon_length" value="0.5"/>
+    <xacro:property name="addon_width" value="0.05"/>
     <!-- links -->
     <link name="car_link"><!--from origin to top-->
@@ -181,4 +183,33 @@
             </geometry>
         </collision>
+    </link>
+    <!-- addon links for support of wx_link -->
+    <link name="addon_Vertical_link">
+        <inertial>
+            <origin xyz="0.0 0.0 ${addon_length/2.0}" rpy="0.0 0.0 0.0"/>
+            <mass value="${little_mass}"/>
+            <inertia ixx="${little_mass}" ixy="0.0" ixz="0.0" iyy="${little_mass}" iyz="0.0" izz="${little_mass}"/>
+        </inertial>
+        <visual>
+            <origin xyz="0.0 0.0 ${addon_length/2.0}" rpy="0.0 0.0 0.0"/>
+            <geometry>
+                <box size="${addon_width} ${addon_width} ${addon_length}"/>
+            </geometry>
+            <material name="purple"/>
+        </visual>
+    </link>
+    <link name="addon_Tilt_link">
+        <inertial>
+            <origin xyz="0.0 0.0 ${addon_length/2.0}" rpy="0.0 0.0 0.0"/>
+            <mass value="${little_mass}"/>
+            <inertia ixx="${little_mass}" ixy="0.0" ixz="0.0" iyy="${little_mass}" iyz="0.0" izz="${little_mass}"/>
+        </inertial>
+        <visual>
+            <origin xyz="0.0 0.0 ${addon_length/2.0}" rpy="0.0 0.0 0.0"/>
+            <geometry>
+                <box size="${addon_width} ${addon_width} ${addon_length}"/>
+            </geometry>
+            <material name="purple"/>
+        </visual>
     </link>
     <!-- joints -->
@@ -225,8 +256,10 @@
         <limit lower="${-PI/2.0}" upper="${PI/2.0}" effort="5.0" velocity="0.5"/>
     </joint>
-    <joint name="littleZ_to_wx" type="fixed">
-        <origin xyz="0.0 0.0 0.0" rpy="0.0 0.0 0.0"/>
-        <parent link="littleZ_link"/>
+    <joint name="addon_Tilt_to_wx" type="continuous">
+        <origin xyz="0.0 0.0 ${addon_length}" rpy="0.0 0.0 0.0"/>
+        <parent link="addon_Tilt_link"/>
         <child link="wx_link"/>
+        <axis xyz="0.0 0.0 1.0"/>
+        <limit effort="5.0" velocity="0.5"/>
     </joint>
     <!-- up and down joints -->
@@ -236,7 +269,7 @@
         <child link="down_link"/>
     </joint>
-    <joint name="littleY_to_up" type="fixed">
+    <joint name="littleZ_to_up" type="fixed">
         <origin xyz="0.0 0.0 0.0" rpy="0.0 0.0 0.0"/>
-        <parent link="littleY_link"/>
+        <parent link="littleZ_link"/>
         <child link="up_link"/>
     </joint>
@@ -254,3 +287,14 @@
     <xacro:sub_link_joint parent_link="up_link" child_link="up_5" height="${up_height}" radius="${up_radius}" beta="290.0" little_width="${little_width}" little_mass="${little_mass}" />
     <xacro:sub_link_joint parent_link="up_link" child_link="up_6" height="${up_height}" radius="${up_radius}" beta="310.0" little_width="${little_width}" little_mass="${little_mass}" />
+    <!--addon joints-->
+    <joint name="littleZ_to_addon_Vertical" type="fixed">
+        <origin xyz="0.0 0.0 0.0" rpy="0.0 0.0 0.0"/>
+        <parent link="littleZ_link"/>
+        <child link="addon_Vertical_link"/>
+    </joint>
+    <joint name="addon_Vertical_to_addon_Tilt" type="fixed">
+        <origin xyz="0.0 0.0 ${addon_length}" rpy="0.0 ${PI/4.0} 0.0"/>
+        <parent link="addon_Vertical_link"/>
+        <child link="addon_Tilt_link"/>
+    </joint>
 </robot>
