Commit message: car to box

File: urdf/parallel_car.gazebo.xacro (robot description, xacro)
@@ -17,4 +17,10 @@
         <material>Gazebo/White</material>
     </gazebo>
+    <gazebo reference="down_link">
+        <material>Gazebo/Grey</material>
+    </gazebo>
+    <gazebo reference="up_link">
+        <material>Gazebo/Orange</material>
+    </gazebo>
     <!-- ros_control plugin -->
     <gazebo>

File: urdf/parallel_car.urdf.xacro (robot description, xacro)
@@ -7,4 +7,5 @@
     <!--xacro properties-->
     <xacro:property name="car_mass" value="20.0"/>
+    <xacro:property name="car_offset" value="0.23"/>
     <xacro:property name="wx_mass" value="5.0"/>
     <xacro:property name="PI" value="3.1415926536"/>
@@ -17,14 +18,14 @@
         <visual>
             <geometry>
-	            <mesh filename="package://parallel_car/meshes/car.STL" />
+                <box size="1 0.5 0.36"/>
      	    </geometry>
             <material name="green"/>
-            <origin rpy="${PI/2.0} 0 ${PI/2.0}" xyz="0 0 0.23"/>
-        </visual>
-        <collision>
-            <geometry>
-	            <mesh filename="package://parallel_car/meshes/car.STL" />
+            <origin rpy="0.0 0.0 0.0" xyz="0 0 0.0"/>
+        </visual>
+        <collision>
+            <geometry>
+                <box size="1 0.5 0.36"/>
      	    </geometry>
-            <origin rpy="${PI/2.0} 0 ${PI/2.0}" xyz="0 0 0.23"/>
+            <origin rpy="0.0 0.0 0.0" xyz="0 0 0.0"/>
         </collision>
         <inertial>
@@ -146,5 +147,5 @@
                 <mesh filename="package://parallel_car/meshes/platform_down.STL" />
             </geometry>
-            <material name="chocolate"/>
+            <material name="grey"/>
         </visual>
         <collision>

Commit message: gazebo control

File: urdf/parallel_car.gazebo.xacro (robot description, xacro)
@@ -23,4 +23,10 @@
         <material>Gazebo/Orange</material>
     </gazebo>
+    <gazebo reference="addon_Vertical_link">
+        <material>Gazebo/Purple</material>
+    </gazebo>
+    <gazebo reference="addon_Tilt_link">
+        <material>Gazebo/Purple</material>
+    </gazebo>
     <!-- ros_control plugin -->
     <gazebo>

File: urdf/parallel_car.transmission.xacro (robot description, xacro)
@@ -55,3 +55,12 @@
         </actuator>
     </transmission>
+    <transmission name="addon_Tilt_to_wx_trans">
+        <type>transmission_interface/SimpleTransmission</type>
+        <joint name="addon_Tilt_to_wx">
+            <hardwareInterface>hardware_interface/PositionJointInterface</hardwareInterface>
+        </joint>
+        <actuator name="addon_Tilt_to_wx_motor">
+            <mechanicalReduction>1</mechanicalReduction>
+        </actuator>
+    </transmission>
 </robot>

Commit message: add support urdf

File: urdf/parallel_car.gazebo.xacro (robot description, xacro)
@@ -36,5 +36,6 @@
         </plugin>
     </gazebo>
-    <gazebo>
+    <!-- with support links and joints, do not need to use planar_move -->
+    <!--gazebo>
         <plugin name="base_controller" filename="libgazebo_ros_planar_move.so">
             <commandTopic>cmd_vel</commandTopic>
@@ -44,4 +45,4 @@
             <robotBaseFrame>car_link</robotBaseFrame>
         </plugin>
-    </gazebo>
+    </gazebo-->
 </robot>

File: urdf/parallel_car.urdf.xacro (robot description, xacro)
@@ -22,4 +22,7 @@
     <xacro:property name="addon_length" value="0.5"/>
     <xacro:property name="addon_width" value="0.05"/>
+    <!-- inlcude support xacro files -->
+    <!-- need to use some xacro properties little_width, little_mass, so include them here-->
+    <xacro:include filename="$(find parallel_car)/urdf/support.urdf.xacro"/>
     <!-- links -->
     <link name="car_link"><!--from origin to top-->
@@ -45,6 +48,6 @@
         <inertial>
             <origin xyz="0.0 0.0 0.0" rpy="0.0 0.0 0.0"/>
-            <mass value="0.01"/>
-            <inertia ixx="0.01" ixy="0.0" ixz="0.0" iyy="0.01" iyz="0.0" izz="0.01"/>
+            <mass value="${little_mass}"/>
+            <inertia ixx="${little_mass}" ixy="0.0" ixz="0.0" iyy="${little_mass}" iyz="0.0" izz="${little_mass}"/>
         </inertial>
         <visual>
@@ -59,6 +62,6 @@
         <inertial>
             <origin xyz="0.0 0.0 0.0" rpy="0.0 0.0 0.0"/>
-            <mass value="0.01"/>
-            <inertia ixx="0.01" ixy="0.0" ixz="0.0" iyy="0.01" iyz="0.0" izz="0.01"/>
+            <mass value="${little_mass}"/>
+            <inertia ixx="${little_mass}" ixy="0.0" ixz="0.0" iyy="${little_mass}" iyz="0.0" izz="${little_mass}"/>
         </inertial>
         <visual>
@@ -73,6 +76,6 @@
         <inertial>
             <origin xyz="0.0 0.0 0.0" rpy="0.0 0.0 0.0"/>
-            <mass value="0.01"/>
-            <inertia ixx="0.01" ixy="0.0" ixz="0.0" iyy="0.01" iyz="0.0" izz="0.01"/>
+            <mass value="${little_mass}"/>
+            <inertia ixx="${little_mass}" ixy="0.0" ixz="0.0" iyy="${little_mass}" iyz="0.0" izz="${little_mass}"/>
         </inertial>
         <visual>
@@ -87,6 +90,6 @@
         <inertial>
             <origin xyz="0.0 0.0 0.0" rpy="0.0 0.0 0.0"/>
-            <mass value="0.01"/>
-            <inertia ixx="0.01" ixy="0.0" ixz="0.0" iyy="0.01" iyz="0.0" izz="0.01"/>
+            <mass value="${little_mass}"/>
+            <inertia ixx="${little_mass}" ixy="0.0" ixz="0.0" iyy="${little_mass}" iyz="0.0" izz="${little_mass}"/>
         </inertial>
         <visual>
@@ -100,6 +103,6 @@
         <inertial>
             <origin xyz="0.0 0.0 0.0" rpy="0.0 0.0 0.0"/>
-            <mass value="0.01"/>
-            <inertia ixx="0.01" ixy="0.0" ixz="0.0" iyy="0.01" iyz="0.0" izz="0.01"/>
+            <mass value="${little_mass}"/>
+            <inertia ixx="${little_mass}" ixy="0.0" ixz="0.0" iyy="${little_mass}" iyz="0.0" izz="${little_mass}"/>
         </inertial>
         <visual>
@@ -113,6 +116,6 @@
         <inertial>
             <origin xyz="0.0 0.0 0.0" rpy="0.0 0.0 0.0"/>
-            <mass value="0.01"/>
-            <inertia ixx="0.01" ixy="0.0" ixz="0.0" iyy="0.01" iyz="0.0" izz="0.01"/>
+            <mass value="${little_mass}"/>
+            <inertia ixx="${little_mass}" ixy="0.0" ixz="0.0" iyy="${little_mass}" iyz="0.0" izz="${little_mass}"/>
         </inertial>
         <visual>

Commit message: add wx rot & gazebo control

File: urdf/parallel_car.gazebo.xacro (robot description, xacro)
@@ -26,7 +26,4 @@
         <material>Gazebo/Purple</material>
     </gazebo>
-    <gazebo reference="addon_Tilt_link">
-        <material>Gazebo/Purple</material>
-    </gazebo>
     <!-- ros_control plugin -->
     <gazebo>

File: urdf/parallel_car.transmission.xacro (robot description, xacro)
@@ -55,12 +55,3 @@
         </actuator>
     </transmission>
-    <transmission name="addon_Tilt_to_wx_trans">
-        <type>transmission_interface/SimpleTransmission</type>
-        <joint name="addon_Tilt_to_wx">
-            <hardwareInterface>hardware_interface/PositionJointInterface</hardwareInterface>
-        </joint>
-        <actuator name="addon_Tilt_to_wx_motor">
-            <mechanicalReduction>1</mechanicalReduction>
-        </actuator>
-    </transmission>
 </robot>

File: urdf/parallel_car.urdf.xacro (robot description, xacro)
@@ -127,5 +127,5 @@
         </visual>
     </link>
-    <link name="wx_link">
+    <link name="wx_visual_link">
         <inertial>
             <origin xyz="0.03 0.0 0.23" rpy="0.0 0.0 0.0"/>
@@ -146,4 +146,17 @@
             </geometry>
         </collision>
+    </link>
+    <link name="wx_link">
+        <inertial>
+            <origin xyz="0.0 0.0 0.0" rpy="0.0 0.0 0.0"/>
+            <mass value="${little_mass}"/>
+            <inertia ixx="${little_mass}" ixy="0.0" ixz="0.0" iyy="${little_mass}" iyz="0.0" izz="${little_mass}"/>
+        </inertial>
+        <visual>
+            <origin xyz="0.0 0.0 0.0" rpy="0.0 0.0 0.0"/>
+            <geometry>
+                <box size="${little_width} ${little_width} ${little_width}"/>
+            </geometry>
+        </visual>
     </link>
     <!-- up and down links -->
@@ -246,7 +259,12 @@
         <limit lower="${-PI/2.0}" upper="${PI/2.0}" effort="50.0" velocity="2.0"/>
     </joint>
-    <joint name="addon_Vertical_to_wx" type="fixed">
+    <joint name="addon_Vertical_to_wx_visual" type="fixed">
         <origin xyz="0.0 0.0 ${addon_length}" rpy="0.0 0.0 0.0"/>
         <parent link="addon_Vertical_link"/>
+        <child link="wx_visual_link"/>
+    </joint>
+    <joint name="wx_visual_to_wx" type="fixed">
+        <origin xyz="0.03 0.0 0.23" rpy="0.0 ${PI/4.0} 0.0"/>
+        <parent link="wx_visual_link"/>
         <child link="wx_link"/>
     </joint>
