Commit message: test with gazebo move and command line succ

File: urdf/support.urdf.xacro (robot description, xacro)
@@ -52,5 +52,5 @@
         <child link="car_link"/>
         <axis xyz="0.0 0.0 1.0"/>
-        <limit lower="-10.0" upper="10.0" effort="100.0" velocity="2.0"/>
+        <limit lower="-10.0" upper="10.0" effort="100.0" velocity="5.0"/>
     </joint>
     <!-- joints end-->
