Commit message: add initial offset in urdf

File: urdf/support.transmission.xacro (robot description, xacro)
@@ -1,10 +1,10 @@
 <?xml version="1.0"?>
 <robot xmlns:xacro="http://www.ros.org/wiki/xacro">
-    <transmission name="world_to_supportX_trans">
+    <transmission name="world_medium_to_supportX_trans">
         <type>transmission_interface/SimpleTransmission</type>
-        <joint name="world_to_supportX">
+        <joint name="world_medium_to_supportX">
             <hardwareInterface>hardware_interface/PositionJointInterface</hardwareInterface>
         </joint>
-        <actuator name="world_to_supportX_motor">
+        <actuator name="world_medium_to_supportX_motor">
             <mechanicalReduction>1</mechanicalReduction>
         </actuator>

File: urdf/support.urdf.xacro (robot description, xacro)
@@ -3,6 +3,22 @@
     <!-- include xacro files -->
     <xacro:include filename="$(find parallel_car)/urdf/support.transmission.xacro"/>
+    <!-- initial position -->
+    <xacro:property name="initial_x" value="0.0"/>
+    <xacro:property name="initial_y" value="-1.5"/>
     <!--links-->
     <link name="world"/>
+    <link name="world_medium_link">
+        <inertial>
+            <origin xyz="0.0 0.0 0.0" rpy="0.0 0.0 0.0"/>
+            <mass value="${little_mass}"/>
+            <inertia ixx="${little_mass}" ixy="0.0" ixz="0.0" iyy="${little_mass}" iyz="0.0" izz="${little_mass}"/>
+        </inertial>
+        <visual>
+            <origin xyz="0.0 0.0 0.0" rpy="0.0 0.0 0.0"/>
+            <geometry>
+                <box size="${little_width} ${little_width} ${little_width}"/>
+            </geometry>
+        </visual>
+    </link>
     <link name="supportX_link">
         <inertial>
@@ -33,7 +49,12 @@
     <!-- links end-->
     <!-- joints -->
-    <joint name="world_to_supportX" type="prismatic">
+    <joint name="world_to_world_medium" type="fixed">
+        <origin xyz="${initial_x} ${initial_y} 0.0" rpy="0.0 0.0 0.0"/>
+        <parent link="world"/>
+        <child link="world_medium_link"/>
+    </joint>
+    <joint name="world_medium_to_supportX" type="prismatic">
         <origin xyz="0.0 0.0 0.0" rpy="0.0 0.0 0.0"/>
-        <parent link="world"/>
+        <parent link="world_medium_link"/>
         <child link="supportX_link"/>
         <axis xyz="1.0 0.0 0.0"/>
