Commit message: add revolute

File: urdf/parallel_car.urdf.xacro (robot description, xacro)
@@ -6,4 +6,5 @@
     <xacro:property name="bar_length" value="1.0"/>
     <xacro:property name="bar_width" value="0.05"/>
+    <xacro:property name="little_width" value="0.001"/>
     <!-- links -->
     <link name="car_link"><!--from origin to top-->
@@ -76,4 +77,52 @@
         </visual>
     </link>
+    <link name="littleX_link">
+        <inertial>
+            <origin xyz="0.0 0.0 0.0" rpy="0.0 0.0 0.0"/>
+            <mass value="0.01"/>
+            <inertia ixx="0.01" ixy="0.0" ixz="0.0" iyy="0.01" iyz="0.0" izz="0.01"/>
+        </inertial>
+        <visual>
+            <origin xyz="0.0 0.0 0.0" rpy="0.0 0.0 0.0"/>
+            <geometry>
+                <box size="${little_width} ${little_width} ${little_width}"/>
+            </geometry>
+            <material name="Chocolate">
+                <color rgba="0.8 0.5 0.125 0.5"/>
+            </material>
+        </visual>
+    </link>
+    <link name="littleY_link">
+        <inertial>
+            <origin xyz="0.0 0.0 0.0" rpy="0.0 0.0 0.0"/>
+            <mass value="0.01"/>
+            <inertia ixx="0.01" ixy="0.0" ixz="0.0" iyy="0.01" iyz="0.0" izz="0.01"/>
+        </inertial>
+        <visual>
+            <origin xyz="0.0 0.0 0.0" rpy="0.0 0.0 0.0"/>
+            <geometry>
+                <box size="${little_width} ${little_width} ${little_width}"/>
+            </geometry>
+            <material name="DarkGreen">
+                <color rgba="0.0 0.5 0.0 0.5"/>
+            </material>
+        </visual>
+    </link>
+    <link name="littleZ_link">
+        <inertial>
+            <origin xyz="0.0 0.0 0.0" rpy="0.0 0.0 0.0"/>
+            <mass value="0.01"/>
+            <inertia ixx="0.01" ixy="0.0" ixz="0.0" iyy="0.01" iyz="0.0" izz="0.01"/>
+        </inertial>
+        <visual>
+            <origin xyz="0.0 0.0 0.0" rpy="0.0 0.0 0.0"/>
+            <geometry>
+                <box size="${little_width} ${little_width} ${little_width}"/>
+            </geometry>
+            <material name="Red">
+                <color rgba="1.0 0.0 0.0 0.5"/>
+            </material>
+        </visual>
+    </link>
     <!-- joints -->
     <joint name="car_to_barX" type="prismatic">
@@ -82,5 +131,5 @@
         <child link="barX_link"/>
         <axis xyz="1.0 0.0 0.0"/>
-        <limit lower="-0.5" upper="0.5" effort="0.5" velocity="0.5"/>
+        <limit lower="-0.5" upper="0.5" effort="5.0" velocity="0.5"/>
     </joint>
     <joint name="barX_to_barY" type="prismatic">
@@ -89,5 +138,5 @@
         <child link="barY_link"/>
         <axis xyz="1.0 0.0 0.0"/>
-        <limit lower="-0.5" upper="0.5" effort="0.5" velocity="0.5"/>
+        <limit lower="-0.5" upper="0.5" effort="5.0" velocity="0.5"/>
     </joint>
     <joint name="barY_to_barZ" type="prismatic">
@@ -96,5 +145,26 @@
         <child link="barZ_link"/>
         <axis xyz="0.0 0.0 1.0"/>
-        <limit lower="-0.5" upper="0.5" effort="0.5" velocity="0.5"/>
+        <limit lower="-0.5" upper="0.5" effort="5.0" velocity="0.5"/>
+    </joint>
+    <joint name="barZ_to_littleX" type="revolute">
+        <origin xyz="0.0 0.0 ${bar_length/2.0}" rpy="0.0 0.0 ${-PI/2.0}"/>
+        <parent link="barZ_link"/>
+        <child link="littleX_link"/>
+        <axis xyz="1.0 0.0 0.0"/>
+        <limit lower="${-PI/2.0}" upper="${PI/2.0}" effort="5.0" velocity="0.5"/>
+    </joint>
+    <joint name="littleX_to_littleY" type="revolute">
+        <origin xyz="0.0 0.0 0.0" rpy="0.0 0.0 ${PI/2.0}"/>
+        <parent link="littleX_link"/>
+        <child link="littleY_link"/>
+        <axis xyz="1.0 0.0 0.0"/>
+        <limit lower="${-PI/2.0}" upper="${PI/2.0}" effort="5.0" velocity="0.5"/>
+    </joint>
+    <joint name="littleY_to_littleZ" type="revolute">
+        <origin xyz="0.0 0.0 0.0" rpy="0.0 0.0 0.0"/>
+        <parent link="littleY_link"/>
+        <child link="littleZ_link"/>
+        <axis xyz="0.0 0.0 1.0"/>
+        <limit lower="${-PI/2.0}" upper="${PI/2.0}" effort="5.0" velocity="0.5"/>
     </joint>
 </robot>

Commit message: add wx

File: urdf/parallel_car.urdf.xacro (robot description, xacro)
@@ -3,8 +3,10 @@
     <!--xacro properties-->
     <xacro:property name="car_mass" value="20.0"/>
+    <xacro:property name="wx_mass" value="5.0"/>
     <xacro:property name="PI" value="3.1415926536"/>
     <xacro:property name="bar_length" value="1.0"/>
     <xacro:property name="bar_width" value="0.05"/>
     <xacro:property name="little_width" value="0.001"/>
+    <xacro:property name="wx_length" value="0.55"/>
     <!-- links -->
     <link name="car_link"><!--from origin to top-->
@@ -26,5 +28,5 @@
         <inertial>
             <mass value="${car_mass}"/>
-            <inertia ixx="1.0" ixy="0.0" ixz="0.0" iyy="1.0" iyz="0.0" izz="1.0" />
+            <inertia ixx="${car_mass}" ixy="0.0" ixz="0.0" iyy="${car_mass}" iyz="0.0" izz="${car_mass}" />
         </inertial>
     </link>
@@ -54,5 +56,5 @@
             <origin xyz="0.0 0.0 0.0" rpy="0.0 0.0 0.0"/>
             <geometry>
-                <box size="${bar_length} ${bar_width} ${bar_width}"/>
+                <box size="${bar_width} ${bar_length} ${bar_width}"/>
             </geometry>
             <material name = "Crimson">
@@ -125,4 +127,26 @@
         </visual>
     </link>
+    <link name="wx_link">
+        <inertial>
+            <origin xyz="0.0 0.0 ${wx_length/2.0}" rpy="0.0 0.0 0.0"/>
+            <mass value="${wx_mass}"/>
+            <inertia ixx="${wx_mass}" ixy="0.0" ixz="0.0" iyy="${wx_mass}" iyz="0.0" izz="${wx_mass}"/>
+        </inertial>
+        <visual>
+            <origin xyz="0.0 0.0 ${wx_length}" rpy="0.0 ${PI} 0.0"/>
+            <geometry>
+                <mesh filename="package://parallel_car/meshes/MZ.STL" />
+            </geometry>
+            <material name="White">
+                <color rgba="1.0 1.0 1.0 0.5"/>
+            </material>
+        </visual>
+        <collision>
+            <origin xyz="0.0 0.0 ${wx_length}" rpy="0.0 0.0 0.0"/>
+            <geometry>
+                <mesh filename="package://parallel_car/meshes/MZ.STL" />
+            </geometry>
+        </collision>
+    </link>
     <!-- joints -->
     <joint name="car_to_barX" type="prismatic">
@@ -134,8 +158,8 @@
     </joint>
     <joint name="barX_to_barY" type="prismatic">
-        <origin xyz="0.0 0.0 ${bar_width}" rpy="0.0 0.0 ${PI/2.0}"/>
+        <origin xyz="0.0 0.0 ${bar_width}" rpy="0.0 0.0 0.0"/>
         <parent link="barX_link"/>
         <child link="barY_link"/>
-        <axis xyz="1.0 0.0 0.0"/>
+        <axis xyz="0.0 1.0 0.0"/>
         <limit lower="-0.5" upper="0.5" effort="5.0" velocity="0.5"/>
     </joint>
@@ -148,5 +172,5 @@
     </joint>
     <joint name="barZ_to_littleX" type="revolute">
-        <origin xyz="0.0 0.0 ${bar_length/2.0}" rpy="0.0 0.0 ${-PI/2.0}"/>
+        <origin xyz="0.0 0.0 ${bar_length/2.0}" rpy="0.0 0.0 0.0"/>
         <parent link="barZ_link"/>
         <child link="littleX_link"/>
@@ -155,8 +179,8 @@
     </joint>
     <joint name="littleX_to_littleY" type="revolute">
-        <origin xyz="0.0 0.0 0.0" rpy="0.0 0.0 ${PI/2.0}"/>
+        <origin xyz="0.0 0.0 0.0" rpy="0.0 0.0 0.0"/>
         <parent link="littleX_link"/>
         <child link="littleY_link"/>
-        <axis xyz="1.0 0.0 0.0"/>
+        <axis xyz="0.0 1.0 0.0"/>
         <limit lower="${-PI/2.0}" upper="${PI/2.0}" effort="5.0" velocity="0.5"/>
     </joint>
@@ -168,3 +192,8 @@
         <limit lower="${-PI/2.0}" upper="${PI/2.0}" effort="5.0" velocity="0.5"/>
     </joint>
+    <joint name="littleZ_to_wx" type="fixed">
+        <origin xyz="0.0 0.0 0.0" rpy="0.0 0.0 0.0"/>
+        <parent link="littleZ_link"/>
+        <child link="wx_link"/>
+    </joint>
 </robot>

Commit message: chg color

File: urdf/parallel_car.urdf.xacro (robot description, xacro)
@@ -4,4 +4,5 @@
     <xacro:include filename="$(find parallel_car)/urdf/parallel_car.gazebo.xacro"/>
     <xacro:include filename="$(find parallel_car)/urdf/parallel_car.transmission.xacro"/>
+    <xacro:include filename="$(find parallel_car)/urdf/materials.xacro"/>
     <!--xacro properties-->
     <xacro:property name="car_mass" value="20.0"/>
@@ -18,7 +19,5 @@
 	            <mesh filename="package://parallel_car/meshes/car.STL" />
      	    </geometry>
-            <material name="ForestGreen">
-                <color rgba="0.15 0.5 0.15 0.5"/>
-            </material>
+            <material name="green"/>
             <origin rpy="${PI/2.0} 0 ${PI/2.0}" xyz="0 0 0.23"/>
         </visual>
@@ -45,7 +44,5 @@
                 <box size="${bar_length} ${bar_width} ${bar_width}"/>
             </geometry>
-            <material name = "Blue">
-                <color rgba = "0.0 0.0 1.0 0.5"/>
-            </material>
+            <material name="blue"/>
         </visual>
     </link>
@@ -61,7 +58,5 @@
                 <box size="${bar_width} ${bar_length} ${bar_width}"/>
             </geometry>
-            <material name = "Crimson">
-                <color rgba="0.8 0.1 0.25 0.5"/>
-            </material>
+            <material name="red"/>
         </visual>
     </link>
@@ -77,7 +72,5 @@
                 <box size="${bar_width} ${bar_width} ${bar_length}"/>
             </geometry>
-            <material name="Yellow">
-                <color rgba="1.0 1.0 0.0 0.5"/>
-            </material>
+            <material name="yellow"/>
         </visual>
     </link>
@@ -93,7 +86,4 @@
                 <box size="${little_width} ${little_width} ${little_width}"/>
             </geometry>
-            <material name="Chocolate">
-                <color rgba="0.8 0.5 0.125 0.5"/>
-            </material>
         </visual>
     </link>
@@ -109,7 +99,4 @@
                 <box size="${little_width} ${little_width} ${little_width}"/>
             </geometry>
-            <material name="DarkGreen">
-                <color rgba="0.0 0.5 0.0 0.5"/>
-            </material>
         </visual>
     </link>
@@ -125,7 +112,4 @@
                 <box size="${little_width} ${little_width} ${little_width}"/>
             </geometry>
-            <material name="Red">
-                <color rgba="1.0 0.0 0.0 0.5"/>
-            </material>
         </visual>
     </link>
@@ -141,7 +125,5 @@
                 <mesh filename="package://parallel_car/meshes/MZ.STL" />
             </geometry>
-            <material name="White">
-                <color rgba="1.0 1.0 1.0 0.5"/>
-            </material>
+            <material name="white"/>
         </visual>
         <collision>
@@ -152,4 +134,5 @@
         </collision>
     </link>
+    <!-- up and down links -->
     <!-- joints -->
     <joint name="car_to_barX" type="prismatic">
@@ -200,3 +183,9 @@
         <child link="wx_link"/>
     </joint>
+    <!-- up and down joints -->
+    <!--joint name="car_to_down" type="fixed">
+        <origin xyz="0.0 0.0 0.18" rpy="0.0 0.0 0.0"/>
+        <parent link="car_link"/>
+        <child link="down_link"/>
+    </joint-->
 </robot>

Commit message: add support control

File: urdf/parallel_car.urdf.xacro (robot description, xacro)
@@ -222,5 +222,5 @@
         <child link="barX_link"/>
         <axis xyz="1.0 0.0 0.0"/>
-        <limit lower="-0.5" upper="0.5" effort="5.0" velocity="0.5"/>
+        <limit lower="-0.5" upper="0.5" effort="50.0" velocity="2.0"/>
     </joint>
     <joint name="barX_to_barY" type="prismatic">
@@ -229,5 +229,5 @@
         <child link="barY_link"/>
         <axis xyz="0.0 1.0 0.0"/>
-        <limit lower="-0.5" upper="0.5" effort="5.0" velocity="0.5"/>
+        <limit lower="-0.5" upper="0.5" effort="50.0" velocity="2.0"/>
     </joint>
     <joint name="barY_to_barZ" type="prismatic">
@@ -236,5 +236,5 @@
         <child link="barZ_link"/>
         <axis xyz="0.0 0.0 1.0"/>
-        <limit lower="-0.5" upper="0.5" effort="5.0" velocity="0.5"/>
+        <limit lower="-0.5" upper="0.5" effort="80.0" velocity="2.0"/>
     </joint>
     <joint name="barZ_to_littleX" type="revolute">

Commit message: add compute optimal alpha

File: urdf/parallel_car.urdf.xacro (robot description, xacro)
@@ -243,5 +243,5 @@
         <child link="littleX_link"/>
         <axis xyz="1.0 0.0 0.0"/>
-        <limit lower="${-PI/2.0}" upper="${PI/2.0}" effort="5.0" velocity="0.5"/>
+        <limit lower="${-PI/2.0}" upper="${PI/2.0}" effort="50.0" velocity="0.5"/>
     </joint>
     <joint name="littleX_to_littleY" type="revolute">
@@ -250,5 +250,5 @@
         <child link="littleY_link"/>
         <axis xyz="0.0 1.0 0.0"/>
-        <limit lower="${-PI/2.0}" upper="${PI/2.0}" effort="5.0" velocity="0.5"/>
+        <limit lower="${-PI/2.0}" upper="${PI/2.0}" effort="50.0" velocity="0.5"/>
     </joint>
     <joint name="littleY_to_littleZ" type="revolute">
@@ -257,5 +257,5 @@
         <child link="littleZ_link"/>
         <axis xyz="0.0 0.0 1.0"/>
-        <limit lower="${-PI/2.0}" upper="${PI/2.0}" effort="5.0" velocity="0.5"/>
+        <limit lower="${-PI/2.0}" upper="${PI/2.0}" effort="50.0" velocity="0.5"/>
     </joint>
     <joint name="addon_Tilt_to_wx" type="continuous">
@@ -264,5 +264,5 @@
         <child link="wx_link"/>
         <axis xyz="0.0 0.0 1.0"/>
-        <limit effort="5.0" velocity="0.5"/>
+        <limit effort="50.0" velocity="0.5"/>
     </joint>
     <!-- up and down joints -->

Commit message: chg world to car height

File: urdf/parallel_car.urdf.xacro (robot description, xacro)
@@ -22,4 +22,5 @@
     <xacro:property name="addon_length" value="0.5"/>
     <xacro:property name="addon_width" value="0.05"/>
+    <xacro:property name="car_height" value="0.36"/>
     <!-- inlcude support xacro files -->
     <!-- need to use some xacro properties little_width, little_mass, so include them here-->
@@ -29,5 +30,5 @@
         <visual>
             <geometry>
-                <box size="1 0.5 0.36"/>
+                <box size="1 0.5 ${car_height}"/>
      	    </geometry>
             <material name="green"/>

File: urdf/support.urdf.xacro (robot description, xacro)
@@ -48,5 +48,5 @@
     </joint>
     <joint name="supportY_to_car" type="continuous">
-        <origin xyz="0.0 0.0 0.0" rpy="0.0 0.0 0.0"/>
+        <origin xyz="0.0 0.0 ${car_height/2.0}" rpy="0.0 0.0 0.0"/>
         <parent link="supportY_link"/>
         <child link="car_link"/>

Commit message: add send one by one

File: urdf/parallel_car.urdf.xacro (robot description, xacro)
@@ -244,5 +244,5 @@
         <child link="littleX_link"/>
         <axis xyz="1.0 0.0 0.0"/>
-        <limit lower="${-PI/2.0}" upper="${PI/2.0}" effort="50.0" velocity="0.5"/>
+        <limit lower="${-PI/2.0}" upper="${PI/2.0}" effort="50.0" velocity="2.0"/>
     </joint>
     <joint name="littleX_to_littleY" type="revolute">
@@ -251,5 +251,5 @@
         <child link="littleY_link"/>
         <axis xyz="0.0 1.0 0.0"/>
-        <limit lower="${-PI/2.0}" upper="${PI/2.0}" effort="50.0" velocity="0.5"/>
+        <limit lower="${-PI/2.0}" upper="${PI/2.0}" effort="50.0" velocity="2.0"/>
     </joint>
     <joint name="littleY_to_littleZ" type="revolute">
@@ -258,5 +258,5 @@
         <child link="littleZ_link"/>
         <axis xyz="0.0 0.0 1.0"/>
-        <limit lower="${-PI/2.0}" upper="${PI/2.0}" effort="50.0" velocity="0.5"/>
+        <limit lower="${-PI/2.0}" upper="${PI/2.0}" effort="50.0" velocity="2.0"/>
     </joint>
     <joint name="addon_Tilt_to_wx" type="continuous">
@@ -265,5 +265,5 @@
         <child link="wx_link"/>
         <axis xyz="0.0 0.0 1.0"/>
-        <limit effort="50.0" velocity="0.5"/>
+        <limit effort="50.0" velocity="2.0"/>
     </joint>
     <!-- up and down joints -->

File: urdf/support.urdf.xacro (robot description, xacro)
@@ -38,5 +38,5 @@
         <child link="supportX_link"/>
         <axis xyz="1.0 0.0 0.0"/>
-        <limit lower="-10.0" upper="10.0" effort="50.0" velocity="5.0"/>
+        <limit lower="-10.0" upper="10.0" effort="100.0" velocity="5.0"/>
     </joint>
     <joint name="supportX_to_supportY" type="prismatic">
@@ -45,5 +45,5 @@
         <child link="supportY_link"/>
         <axis xyz="0.0 1.0 0.0"/>
-        <limit lower="-10.0" upper="10.0" effort="50.0" velocity="5.0"/>
+        <limit lower="-10.0" upper="10.0" effort="100.0" velocity="5.0"/>
     </joint>
     <joint name="supportY_to_car" type="continuous">
@@ -52,5 +52,5 @@
         <child link="car_link"/>
         <axis xyz="0.0 0.0 1.0"/>
-        <limit lower="-10.0" upper="10.0" effort="50.0" velocity="2.0"/>
+        <limit lower="-10.0" upper="10.0" effort="100.0" velocity="2.0"/>
     </joint>
     <!-- joints end-->

Commit message: chg urdf model

File: urdf/parallel_car.urdf.xacro (robot description, xacro)
@@ -21,5 +21,5 @@
     <xacro:property name="little_mass" value="0.01"/>
     <xacro:property name="addon_length" value="0.5"/>
-    <xacro:property name="addon_width" value="0.05"/>
+    <xacro:property name="addon_width" value="0.01"/>
     <xacro:property name="car_height" value="0.36"/>
     <!-- inlcude support xacro files -->
@@ -129,10 +129,10 @@
     <link name="wx_link">
         <inertial>
-            <origin xyz="0.0 0.0 ${wx_length/2.0}" rpy="0.0 0.0 0.0"/>
+            <origin xyz="0.03 0.0 0.23" rpy="0.0 0.0 0.0"/>
             <mass value="${wx_mass}"/>
             <inertia ixx="${wx_mass}" ixy="0.0" ixz="0.0" iyy="${wx_mass}" iyz="0.0" izz="${wx_mass}"/>
         </inertial>
         <visual>
-            <origin xyz="0.0 0.0 ${wx_length}" rpy="0.0 ${PI} 0.0"/>
+            <origin xyz="0.05 0.0 0.25" rpy="${3.0*PI/4.0} 0.0 ${-PI/2.0}"/>
             <geometry>
                 <mesh filename="package://parallel_car/meshes/MZ.STL" />
@@ -141,5 +141,5 @@
         </visual>
         <collision>
-            <origin xyz="0.0 0.0 ${wx_length}" rpy="0.0 0.0 0.0"/>
+            <origin xyz="0.05 0.0 0.25" rpy="0.0 0.0 0.0"/>
             <geometry>
                 <mesh filename="package://parallel_car/meshes/MZ.STL" />
@@ -190,18 +190,4 @@
     <!-- addon links for support of wx_link -->
     <link name="addon_Vertical_link">
-        <inertial>
-            <origin xyz="0.0 0.0 ${addon_length/2.0}" rpy="0.0 0.0 0.0"/>
-            <mass value="${little_mass}"/>
-            <inertia ixx="${little_mass}" ixy="0.0" ixz="0.0" iyy="${little_mass}" iyz="0.0" izz="${little_mass}"/>
-        </inertial>
-        <visual>
-            <origin xyz="0.0 0.0 ${addon_length/2.0}" rpy="0.0 0.0 0.0"/>
-            <geometry>
-                <box size="${addon_width} ${addon_width} ${addon_length}"/>
-            </geometry>
-            <material name="purple"/>
-        </visual>
-    </link>
-    <link name="addon_Tilt_link">
         <inertial>
             <origin xyz="0.0 0.0 ${addon_length/2.0}" rpy="0.0 0.0 0.0"/>
@@ -260,10 +246,8 @@
         <limit lower="${-PI/2.0}" upper="${PI/2.0}" effort="50.0" velocity="2.0"/>
     </joint>
-    <joint name="addon_Tilt_to_wx" type="continuous">
+    <joint name="addon_Vertical_to_wx" type="fixed">
         <origin xyz="0.0 0.0 ${addon_length}" rpy="0.0 0.0 0.0"/>
-        <parent link="addon_Tilt_link"/>
+        <parent link="addon_Vertical_link"/>
         <child link="wx_link"/>
-        <axis xyz="0.0 0.0 1.0"/>
-        <limit effort="50.0" velocity="2.0"/>
     </joint>
     <!-- up and down joints -->
@@ -297,8 +281,3 @@
         <child link="addon_Vertical_link"/>
     </joint>
-    <joint name="addon_Vertical_to_addon_Tilt" type="fixed">
-        <origin xyz="0.0 0.0 ${addon_length}" rpy="0.0 ${PI/4.0} 0.0"/>
-        <parent link="addon_Vertical_link"/>
-        <child link="addon_Tilt_link"/>
-    </joint>
 </robot>

Commit message: chg model

File: urdf/parallel_car.urdf.xacro (robot description, xacro)
@@ -147,4 +147,17 @@
         </collision>
     </link>
+    <link name="wx_medium_link">
+        <inertial>
+            <origin xyz="0.0 0.0 0.0" rpy="0.0 0.0 0.0"/>
+            <mass value="${little_mass}"/>
+            <inertia ixx="${little_mass}" ixy="0.0" ixz="0.0" iyy="${little_mass}" iyz="0.0" izz="${little_mass}"/>
+        </inertial>
+        <visual>
+            <origin xyz="0.0 0.0 0.0" rpy="0.0 0.0 0.0"/>
+            <geometry>
+                <box size="${little_width} ${little_width} ${little_width}"/>
+            </geometry>
+        </visual>
+    </link>
     <link name="wx_link">
         <inertial>
@@ -264,7 +277,12 @@
         <child link="wx_visual_link"/>
     </joint>
-    <joint name="wx_visual_to_wx" type="fixed">
+    <joint name="wx_visual_to_wx_medium" type="fixed">
         <origin xyz="0.03 0.0 0.23" rpy="0.0 ${PI/4.0} 0.0"/>
         <parent link="wx_visual_link"/>
+        <child link="wx_medium_link"/>
+    </joint>
+    <joint name="wx_medium_to_wx" type="fixed">
+        <origin xyz="0.0 0.0 0.0" rpy="0.0 0.0 ${-PI/2.0}"/>
+        <parent link="wx_medium_link"/>
         <child link="wx_link"/>
     </joint>

Commit message: chg trans limit&test with single line succ

File: urdf/parallel_car.urdf.xacro (robot description, xacro)
@@ -235,5 +235,5 @@
         <child link="barX_link"/>
         <axis xyz="1.0 0.0 0.0"/>
-        <limit lower="-0.5" upper="0.5" effort="50.0" velocity="2.0"/>
+        <limit lower="-1.0" upper="1.0" effort="50.0" velocity="2.0"/>
     </joint>
     <joint name="barX_to_barY" type="prismatic">
@@ -242,5 +242,5 @@
         <child link="barY_link"/>
         <axis xyz="0.0 1.0 0.0"/>
-        <limit lower="-0.5" upper="0.5" effort="50.0" velocity="2.0"/>
+        <limit lower="-1.0" upper="1.0" effort="50.0" velocity="2.0"/>
     </joint>
     <joint name="barY_to_barZ" type="prismatic">
@@ -249,5 +249,5 @@
         <child link="barZ_link"/>
         <axis xyz="0.0 0.0 1.0"/>
-        <limit lower="-0.5" upper="0.5" effort="80.0" velocity="2.0"/>
+        <limit lower="-1.0" upper="1.0" effort="80.0" velocity="2.0"/>
     </joint>
     <joint name="barZ_to_littleX" type="revolute">

Commit message: reduce bar length

File: urdf/parallel_car.urdf.xacro (robot description, xacro)
@@ -11,5 +11,5 @@
     <xacro:property name="wx_mass" value="5.0"/>
     <xacro:property name="PI" value="3.1415926536"/>
-    <xacro:property name="bar_length" value="1.0"/>
+    <xacro:property name="bar_length" value="0.5"/>
     <xacro:property name="bar_width" value="0.05"/>
     <xacro:property name="little_width" value="0.001"/>
@@ -20,5 +20,5 @@
     <xacro:property name="up_height" value="0.05"/>
     <xacro:property name="little_mass" value="0.01"/>
-    <xacro:property name="addon_length" value="0.5"/>
+    <xacro:property name="addon_length" value="0.4"/>
     <xacro:property name="addon_width" value="0.01"/>
     <xacro:property name="car_height" value="0.36"/>
