Commit message: reduce bar length to 0.4

File: urdf/parallel_car.urdf.xacro (robot description, xacro)
@@ -11,11 +11,11 @@
     <xacro:property name="wx_mass" value="5.0"/>
     <xacro:property name="PI" value="3.1415926536"/>
-    <xacro:property name="bar_length" value="0.5"/>
+    <xacro:property name="bar_length" value="0.4"/>
     <xacro:property name="bar_width" value="0.05"/>
     <xacro:property name="little_width" value="0.001"/>
     <xacro:property name="wx_length" value="0.55"/>
-    <xacro:property name="down_radius" value="0.2"/>
+    <xacro:property name="down_radius" value="0.21"/>
     <xacro:property name="down_height" value="0.075"/>
-    <xacro:property name="up_radius" value="0.1"/>
+    <xacro:property name="up_radius" value="0.125"/>
     <xacro:property name="up_height" value="0.05"/>
     <xacro:property name="little_mass" value="0.01"/>

Commit message: chg car stl

File: urdf/parallel_car.urdf.xacro (robot description, xacro)
@@ -30,14 +30,14 @@
         <visual>
             <geometry>
-                <box size="1 0.5 ${car_height}"/>
+                <mesh filename="package://parallel_car/meshes/car.STL" />
      	    </geometry>
             <material name="green"/>
-            <origin rpy="0.0 0.0 0.0" xyz="0 0 0.0"/>
+            <origin rpy="${PI/2.0} 0.0 0.0" xyz="0 0 -0.12"/>
         </visual>
         <collision>
             <geometry>
-                <box size="1 0.5 0.36"/>
+                <mesh filename="package://parallel_car/meshes/car.STL" />
      	    </geometry>
-            <origin rpy="0.0 0.0 0.0" xyz="0 0 0.0"/>
+            <origin rpy="${PI/2.0} 0.0 0.0" xyz="0 0 -0.12"/>
         </collision>
         <inertial>

Commit message: chg wx pose

File: urdf/parallel_car.urdf.xacro (robot description, xacro)
@@ -129,10 +129,10 @@
     <link name="wx_visual_link">
         <inertial>
-            <origin xyz="0.03 0.0 0.23" rpy="0.0 0.0 0.0"/>
+            <origin xyz="0.0 0.0 0.0" rpy="${110.0/180.0*PI} 0.0 ${-PI/2.0}"/>
             <mass value="${wx_mass}"/>
             <inertia ixx="${wx_mass}" ixy="0.0" ixz="0.0" iyy="${wx_mass}" iyz="0.0" izz="${wx_mass}"/>
         </inertial>
         <visual>
-            <origin xyz="0.05 0.0 0.25" rpy="${3.0*PI/4.0} 0.0 ${-PI/2.0}"/>
+            <origin xyz="0.0 0.0 0.0" rpy="${110.0/180.0*PI} 0.0 ${-PI/2.0}"/>
             <geometry>
                 <mesh filename="package://parallel_car/meshes/MZ.STL" />
@@ -141,5 +141,5 @@
         </visual>
         <collision>
-            <origin xyz="0.05 0.0 0.25" rpy="0.0 0.0 0.0"/>
+            <origin xyz="0.0 0.0 0.0" rpy="${110.0/180.0*PI} 0.0 ${-PI/2.0}"/>
             <geometry>
                 <mesh filename="package://parallel_car/meshes/MZ.STL" />
@@ -213,19 +213,4 @@
             </geometry>
         </collision>
-    </link>
-    <!-- addon links for support of wx_link -->
-    <link name="addon_Vertical_link">
-        <inertial>
-            <origin xyz="0.0 0.0 ${addon_length/2.0}" rpy="0.0 0.0 0.0"/>
-            <mass value="${little_mass}"/>
-            <inertia ixx="${little_mass}" ixy="0.0" ixz="0.0" iyy="${little_mass}" iyz="0.0" izz="${little_mass}"/>
-        </inertial>
-        <visual>
-            <origin xyz="0.0 0.0 ${addon_length/2.0}" rpy="0.0 0.0 0.0"/>
-            <geometry>
-                <box size="${addon_width} ${addon_width} ${addon_length}"/>
-            </geometry>
-            <material name="purple"/>
-        </visual>
     </link>
     <!-- joints -->
@@ -272,11 +257,11 @@
         <limit lower="${-PI/2.0}" upper="${PI/2.0}" effort="50.0" velocity="2.0"/>
     </joint>
-    <joint name="addon_Vertical_to_wx_visual" type="fixed">
-        <origin xyz="0.0 0.0 ${addon_length}" rpy="0.0 0.0 0.0"/>
-        <parent link="addon_Vertical_link"/>
+    <joint name="littleZ_to_wx_visual" type="fixed">
+        <origin xyz="0.35 0.0 0.25" rpy="0.0 0.0 0.0"/>
+        <parent link="littleZ_link"/>
         <child link="wx_visual_link"/>
     </joint>
     <joint name="wx_visual_to_wx_medium" type="fixed">
-        <origin xyz="0.03 0.0 0.23" rpy="0.0 ${PI/4.0} 0.0"/>
+        <origin xyz="-0.1 0.0 -0.065" rpy="0.0 ${70.0/180.0*PI} 0.0"/>
         <parent link="wx_visual_link"/>
         <child link="wx_medium_link"/>
@@ -311,9 +296,3 @@
     <xacro:sub_link_joint parent_link="up_link" child_link="up_5" height="${up_height}" radius="${up_radius}" beta="290.0" little_width="${little_width}" little_mass="${little_mass}" />
     <xacro:sub_link_joint parent_link="up_link" child_link="up_6" height="${up_height}" radius="${up_radius}" beta="310.0" little_width="${little_width}" little_mass="${little_mass}" />
-    <!--addon joints-->
-    <joint name="littleZ_to_addon_Vertical" type="fixed">
-        <origin xyz="0.0 0.0 0.0" rpy="0.0 0.0 0.0"/>
-        <parent link="littleZ_link"/>
-        <child link="addon_Vertical_link"/>
-    </joint>
 </robot>
